Commit message: update

File: src/bxi_rl_controller_ros2_example/resources/elf3_dof29/urdf/elf3.urdf (robot description, URDF)
Before this commit: robot elf3, 30 links, 29 joints
Links:
- link torso_link: mass 8.0753 -> 12.004
Joints:
- joint l_ankle_x_joint: limit lower=-0.34907 upper=0.34907 effort=15 velocity=20 -> lower=-0.34907 upper=0.34907 effort=20 velocity=20
- joint l_ankle_y_joint: limit lower=-0.87266 upper=0.7854 effort=40 velocity=20 -> lower=-0.87266 upper=0.7854 effort=50 velocity=20
- joint r_ankle_x_joint: limit lower=-0.34907 upper=0.34907 effort=15 velocity=20 -> lower=-0.34907 upper=0.34907 effort=20 velocity=20
- joint r_ankle_y_joint: limit lower=-0.87266 upper=0.7854 effort=40 velocity=20 -> lower=-0.87266 upper=0.7854 effort=50 velocity=20
