Commit message: 更新框架版本

File: src/bxi_rl_controller_ros2_example/resources/elf3_dof31/urdf/elf3.urdf (robot description, URDF)
Before this commit: robot elf3, 35 links, 34 joints
Links:
- added link torso_front_bottom_d435i_link
Joints:
- added joint torso_front_bottom_d435i_joint: type fixed, parent torso_link, child torso_front_bottom_d435i_link, origin xyz=0.1152 0.0175 -0.1358 rpy=-2.7925 0 -1.5708, axis 0 0 0
- joint d435i_joint: origin xyz=0.067 0 -0.048 rpy=-1.5708 0 -1.5708 -> xyz=0.0628 0.0175 -0.048 rpy=-1.5708 0 -1.5708
